Commit message: fixed teleop commands and directions moved

File: src/vehicle_bringup/urdfs/urdf/basic_robot.urdf (robot description, URDF)
Before this commit: robot two_wheel_robot, 5 links, 4 joints
Joints:
- joint left_wheel_joint: axis 0 0 1 -> 0 0 -1
- joint right_wheel_joint: axis 0 0 1 -> 0 0 -1

Commit message: made basic robot slimmer

File: src/vehicle_bringup/urdfs/urdf/basic_robot.urdf (robot description, URDF)
Before this commit: robot two_wheel_robot, 5 links, 4 joints
Links:
- link base_link: geometry collision box size=0.4 0.25 0.2; visual box size=0.4 0.25 0.2
Joints:
- joint left_wheel_joint: origin xyz=-0.1 -0.175 0.0 rpy=1.5708 0.0 0.0 -> xyz=-0.1 -0.15 0.0 rpy=1.5708 0.0 0.0
- joint right_wheel_joint: origin xyz=-0.1 0.175 0.0 rpy=1.5708 0.0 0.0 -> xyz=-0.1 0.15 0.0 rpy=1.5708 0.0 0.0

Commit message: made robot smaller

File: src/vehicle_bringup/urdfs/urdf/basic_robot.urdf (robot description, URDF)
Before this commit: robot two_wheel_robot, 5 links, 4 joints
Links:
- link base_link: mass 5.0 -> 3.0; geometry collision box size=0.3 0.15 0.2; visual box size=0.3 0.15 0.2
- link left_wheel: mass 0.5 -> 0.3; geometry collision cylinder length=0.04 radius=0.05; visual cylinder length=0.04 radius=0.05
- link right_wheel: mass 0.5 -> 0.3; geometry collision cylinder length=0.04 radius=0.05; visual cylinder length=0.04 radius=0.05
Joints:
- joint caster_wheel_joint: origin xyz=0.15 0.0 -0.05 rpy=0 0 0 -> xyz=0.1125 0.0 -0.05 rpy=0 0 0
- joint left_wheel_joint: origin xyz=-0.1 -0.15 0.0 rpy=1.5708 0.0 0.0 -> xyz=-0.075 -0.0875 -0.05 rpy=1.5708 0.0 0.0
- joint right_wheel_joint: origin xyz=-0.1 0.15 0.0 rpy=1.5708 0.0 0.0 -> xyz=-0.075 0.0875 -0.05 rpy=1.5708 0.0 0.0
